Commit message: adapt description for roomba600+tablet+lidar

File: roomblock_description/robots/roomblock.urdf.xacro (robot description, xacro)
@@ -20,5 +20,5 @@
       <origin xyz="0 0 0" rpy="0 0 0" />
       <geometry>
-	<mesh filename="package://roomblock_description/meshes/block.dae"/>
+	      <mesh filename="package://roomblock_description/meshes/block.dae"/>
       </geometry>
       <material name="Grey" />
